File: 119_INTELLIGENT_SENSOR_BOARD/119_02v2_INTELLIGENT_SENSOR_BOARD.brd (EAGLE design)
At the start: 14.6 x 37.5 mm, 14 parts

Commit message: Formed new documentation
Split manual into datasheet, library and notes... added a few more ISC library header defines
Parts:
- removed CONN_GND, CONN_UPDI, CONN_VDD: TPB1,27, testpad:B1,27
- removed V_SEL: (no value), SparkFun-Connectors:1X03
- added 3V3, 3V3BRD, 5V, 5VBRD, LNK: JUMPER-SMT_2_NO_SILK, SparkFun-Jumpers:SMT-JUMPER_2_NO_SILK
Connections:
- new net 3V3_BRD: 3V3BRD.1, LNK.1, SENSOR_BOARD.14
- new net 5V_BRD: 5VBRD.1, LNK.2, SENSOR_BOARD.13
- net 3V3: now also 3V3BRD.2, 5V.2; no longer SENSOR_BOARD.14, V_SEL.1
- net 5V: now also 3V3.2, 5VBRD.2; no longer SENSOR_BOARD.13, V_SEL.3
- net GND: no longer CONN_GND.TP
- net UPDI: no longer CONN_UPDI.TP
- net VDD: now also 3V3.1, 5V.1; no longer CONN_VDD.TP, V_SEL.2
Routing:
- net 5V_BRD: track 0.00 -> 7.65 mm
- net 3V3_BRD: track 0.00 -> 6.12 mm
- net 5V: track 12.3 -> 6.23 mm
- net 3V3: track 12.7 -> 6.74 mm
- net UPDI: track 28.5 -> 24.1 mm
- net GND: track 54.6 -> 50.2 mm
- net VDD: track 43.7 -> 43.4 mm, vias 1 -> 2
